File: board/bleriot-rs485.kicad_pcb (KiCad board)
At the start: 2 copper layers, 40 x 42 mm, 21 parts, among them J3 POWER, J4 RS485, U1 LM1117MP-3.3, U4 ST3485EBDR, U5 PAN2110P0AA, U6 PY32F030F1xPx, X2 SWD, Y2 16MHz

Commit message: Update board configuration and component footprints
- Changed the active layer in the KiCad project file from 0 to 5 for improved layout management.
- Updated silk overlap parameters in the project file to correct values for better design accuracy.
- Added a new starved thermal entry in the project file to enhance thermal performance.
- Replaced the footprint for a connector in the schematic from Phoenix MC series to MSTB series for better compatibility.
- Updated another connector footprint in the schematic to the MSTB series for consistency and improved design.
- Updated submodule reference for hw-kicad to the latest commit for up-to-date hardware support.
Parts:
- J3: footprint Connector_Phoenix_MC:PhoenixContact_MC_1,5_2-G-3.5_1x02_P3.50mm_Horizontal -> Connector_Phoenix_MSTB:PhoenixContact_MSTBA_2,5_2-G_1x02_P5.00mm_Horizontal
- J4: footprint Connector_Phoenix_MC:PhoenixContact_MC_1,5_3-G-3.5_1x03_P3.50mm_Horizontal -> Connector_Phoenix_MSTB:PhoenixContact_MSTBA_2,5_3-G_1x03_P5.00mm_Horizontal
- moved X2 17.3 mm to (166.5, 46.4), turned to 180 degrees
- moved J4 2.41 mm to (147.5, 60.2)
- moved J3 1.97 mm to (170.5, 60.2)
Routing:
- net Net-(U6-PA14): track 12.4 -> 21.8 mm, vias 1 -> 0
- net Net-(U6-PA13): track 16.6 -> 21.9 mm, vias 1 -> 0
- net /RS485_A: track 22.9 -> 18.6 mm
- net +5V: track 19.2 -> 16.3 mm
- net /RS485_B: track 26.7 -> 24.0 mm
- net GND: vias 51 -> 48
Other:
- board text added: "bleriot-rs485 v1.2 drake.cz"
- board text removed: "bleriot-rs485 v1.1 drake.cz"
