File: board/bleriot-rs485.kicad_sch (KiCad schematic)
At the start: 21 parts, among them J3 POWER, J4 RS485, U1 LM1117MP-3.3, U4 ST3485EBDR, U5 PAN2110P0AA, U6 PY32F030F1xPx, X2 SWD, Y2 16MHz

Commit message: Update board configuration and component footprints
- Changed the active layer in the KiCad project file from 0 to 5 for improved layout management.
- Updated silk overlap parameters in the project file to correct values for better design accuracy.
- Added a new starved thermal entry in the project file to enhance thermal performance.
- Replaced the footprint for a connector in the schematic from Phoenix MC series to MSTB series for better compatibility.
- Updated another connector footprint in the schematic to the MSTB series for consistency and improved design.
- Updated submodule reference for hw-kicad to the latest commit for up-to-date hardware support.
Parts:
- J3: footprint Connector_Phoenix_MC:PhoenixContact_MC_1,5_2-G-3.5_1x02_P3.50mm_Horizontal -> Connector_Phoenix_MSTB:PhoenixContact_MSTBA_2,5_2-G_1x02_P5.00mm_Horizontal
- J4: footprint Connector_Phoenix_MC:PhoenixContact_MC_1,5_3-G-3.5_1x03_P3.50mm_Horizontal -> Connector_Phoenix_MSTB:PhoenixContact_MSTBA_2,5_3-G_1x03_P5.00mm_Horizontal
Changed lines of the file:
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@@
 			)
 		)
-		(property "Footprint" "Connector_Phoenix_MC:PhoenixContact_MC_1,5_3-G-3.5_1x03_P3.50mm_Horizontal"
+		(property "Footprint" "Connector_Phoenix_MSTB:PhoenixContact_MSTBA_2,5_3-G_1x03_P5.00mm_Horizontal"
 			(at 35.56 114.3 0)
 			(hide yes)
@@
 			)
 		)
-		(property "Footprint" "Connector_Phoenix_MC:PhoenixContact_MC_1,5_2-G-3.5_1x02_P3.50mm_Horizontal"
+		(property "Footprint" "Connector_Phoenix_MSTB:PhoenixContact_MSTBA_2,5_2-G_1x02_P5.00mm_Horizontal"
 			(at 34.29 135.89 0)
 			(hide yes)
